Commit message: generalize config and interfaces

File: description/ros2_control/example.ros2_control.xacro (robot description, xacro)
@@ -1,12 +1,20 @@
 <?xml version="1.0"?>
 <robot xmlns:xacro="http://www.ros.org/wiki/xacro">
-    <xacro:macro name="example_ws_ros2_control" params="name prefix">
+    <xacro:macro name="example_ws_ros2_control"
+                 params="name prefix port:=/dev/ttyACM0 baudrate:=1000000">
         <ros2_control name="${name}" type="system">
             <hardware>
                 <plugin>waveshare_servos/WaveshareServos</plugin>
-                <param name="example_param_hw_start_duration_sec">0</param>
-                <param name="example_param_hw_stop_duration_sec">3.0</param>
-                <param name="example_param_hw_slowdown">100</param>
+                <param name="port">${port}</param>
+                <param name="baudrate">${baudrate}</param>
+                <!-- Optional, shown with their defaults and deliberately left out so this example
+                     exercises them -
+                     io_timeout_ms 20, ping_attempts 3, max_read_fails 50,
+                     allow_missing_servos false, protocol sms_sts, encoder_steps 4096,
+                     current_per_count_a 0.006, torque_constant_nm_per_a 0.8825985 -->
             </hardware>
+            <!-- State interfaces are free-form - declare any subset of position, velocity,
+                 effort, current, voltage, temperature, load and status, in any order. `torque` is
+                 a deprecated alias of `effort` that keeps reporting kg cm instead of N m. -->
             <joint name="${prefix}joint1">
                 <param name="id">1</param>
@@ -23,5 +31,5 @@
                 <state_interface name="position"/>
                 <state_interface name="velocity"/>
-                <state_interface name="torque"/>
+                <state_interface name="effort"/>
                 <state_interface name="temperature"/>
             </joint>
@@ -40,5 +48,5 @@
                 <state_interface name="position"/>
                 <state_interface name="velocity"/>
-                <state_interface name="torque"/>
+                <state_interface name="effort"/>
                 <state_interface name="temperature"/>
             </joint>
@@ -52,5 +60,28 @@
                 <state_interface name="position"/>
                 <state_interface name="velocity"/>
-                <state_interface name="torque"/>
+                <state_interface name="effort"/>
+                <state_interface name="temperature"/>
+            </joint>
+            <!-- The second wheel, id 4, the same shape as joint3 - the example declares four
+                 joints because the reference bench carries four servos (ids 1-4), and a
+                 three-joint example on a four-servo bus leaves one servo unread and unwritten.
+                 A mirrored wheel pair is what `inverted` exists for - the right-hand wheel of a
+                 differential drive would add a param inverted of true, which flips its two
+                 command interfaces together with its position, velocity and load states, so that
+                 one positive velocity drives the pair forward. It is deliberately left off here,
+                 because the URDF beside this file is a serial chain rather than a mirrored pair,
+                 so an inverted joint4 would spin its servo opposite to the model RViz draws, and
+                 this file is what a new user copies first. See the bench description under
+                 test/hil/descriptions for `inverted` exercised on hardware. -->
+            <joint name="${prefix}joint4">
+                <param name="id">4</param>
+                <param name="type">vel</param>
+                <command_interface name="velocity">
+                    <param name="min">-9.2</param>
+                    <param name="max">9.2</param>
+                </command_interface>
+                <state_interface name="position"/>
+                <state_interface name="velocity"/>
+                <state_interface name="effort"/>
                 <state_interface name="temperature"/>
             </joint>

File: description/urdf/example.urdf.xacro (robot description, xacro)
@@ -62,4 +62,22 @@
         </visual>
     </link>
+    <!-- The second wheel. Every joint of the ros2_control block has to exist here too, so joint4
+         gets a link of its own. -->
+    <joint name="joint4" type="continuous">
+        <axis xyz="0 0 1"/>
+        <limit effort="1000.0" lower="-3.14" upper="3.14" velocity="1.0"/>
+        <origin xyz="0 0 0.1"/>
+        <parent link="link4"/>
+        <child link="link5"/>
+    </joint>
+    <link name="link5">
+        <visual>
+            <origin xyz="0 0 0.05"/>
+            <geometry>
+                <cylinder length="0.1" radius="0.1"/>
+            </geometry>
+            <material name="white"/>
+        </visual>
+    </link>
     <xacro:include filename="$(find waveshare_servos)/description/ros2_control/example.ros2_control.xacro"/>
     <xacro:example_ws_ros2_control name="example_ws_ros2_control" prefix="$(arg prefix)"/>

Commit message: examples, launch, config

File: description/ros2_control/example.ros2_control.xacro (robot description, xacro)
@@ -2,5 +2,12 @@
 <robot xmlns:xacro="http://www.ros.org/wiki/xacro">
     <xacro:macro name="example_ws_ros2_control"
-                 params="name prefix port:=/dev/ttyACM0 baudrate:=1000000">
+                 params="name port:=/dev/ttyACM0 baudrate:=1000000 use_mock_hardware:=false">
+        <!-- use_mock_hardware accepts true, false, 1 or 0, in any case and with any surrounding
+             space. The list lookup is deliberate: an unrecognised spelling raises inside xacro and
+             aborts the render with exit 2 ("'yes' is not in list"), which aborts the launch. A
+             plain string comparison against 'true' would treat use_mock_hardware:=yes as false and
+             quietly open the real serial port instead. -->
+        <xacro:property name="mock"
+            value="${['false', '0', 'true', '1'].index(str(use_mock_hardware).strip().lower()) >= 2}"/>
         <!-- Optional, ros2_control 4.48 - read and write the hardware at its own rate, and/or on
              its own thread. Both are ATTRIBUTES of this element, not <param> children of
@@ -20,18 +27,43 @@
         <ros2_control name="${name}" type="system">
             <hardware>
-                <plugin>waveshare_servos/WaveshareServos</plugin>
-                <param name="port">${port}</param>
-                <param name="baudrate">${baudrate}</param>
-                <!-- Optional, shown with their defaults and deliberately left out so this example
-                     exercises them -
-                     io_timeout_ms 5, ping_attempts 3, max_read_fails 50,
-                     allow_missing_servos false, protocol sms_sts, feedback_mode auto,
-                     encoder_steps 4096, current_per_count_a 0.006,
-                     torque_constant_nm_per_a 0.8825985 -->
+                <!-- use_mock_hardware:=true swaps the driver for ros2_control's own loopback
+                     simulator, which ships inside hardware_interface, opens no serial port and
+                     mirrors every command straight back into its matching state. The four <joint>
+                     blocks below are shared verbatim with the real driver: GenericSystem ignores
+                     the id/type/offset params it does not know, and a state interface with no
+                     command interface (effort, temperature) simply reads a constant 0.0. Two mock
+                     behaviours are not bugs: a velocity-commanded joint's position state never
+                     advances, so joint3 and joint4 stand still in RViz and the diff_drive odometry
+                     stays at zero; and nothing validates port, baudrate or id, so a green mock run
+                     says nothing about your wiring. The obvious cure for the frozen wheel position
+                     - the calculate_dynamics param - is a trap: it rejects any joint claiming two
+                     of position/velocity/acceleration, which is exactly what
+                     joint_trajectory_position_controller does to joint1 and joint2, and that
+                     controller then fails to activate. Do not add it. -->
+                <xacro:if value="${mock}">
+                    <plugin>mock_components/GenericSystem</plugin>
+                </xacro:if>
+                <xacro:unless value="${mock}">
+                    <plugin>waveshare_servos/WaveshareServos</plugin>
+                    <param name="port">${port}</param>
+                    <param name="baudrate">${baudrate}</param>
+                    <!-- Optional, shown with their defaults and deliberately left out so this
+                         example exercises them -
+                         io_timeout_ms 5, ping_attempts 3, max_read_fails 50,
+                         allow_missing_servos false, protocol sms_sts, feedback_mode auto,
+                         encoder_steps 4096, current_per_count_a 0.006,
+                         torque_constant_nm_per_a 0.8825985 -->
+                </xacro:unless>
             </hardware>
             <!-- State interfaces are free-form - declare any subset of position, velocity,
                  effort, current, voltage, temperature, load and status, in any order. `torque` is
-                 a deprecated alias of `effort` that keeps reporting kg cm instead of N m. -->
-            <joint name="${prefix}joint1">
+                 a deprecated alias of `effort` that keeps reporting kg cm instead of N m.
+                 The min/max below and the <limit> tags in the URDF beside this file are MERGED,
+                 most-restrictive-wins, so keep the two numerically identical: whichever is tighter
+                 is what the framework enforces, and a disagreement makes the description behave
+                 differently depending on a controller-manager flag. They only bite when the
+                 controller manager runs with enforce_command_limits: true; this example ships with
+                 it off, and the driver clamps position commands to these same values on its own. -->
+            <joint name="joint1">
                 <param name="id">1</param>
                 <param name="type">pos</param>
@@ -50,5 +82,5 @@
                 <state_interface name="temperature"/>
             </joint>
-            <joint name="${prefix}joint2">
+            <joint name="joint2">
                 <param name="id">2</param>
                 <param name="type">pos</param>
@@ -67,5 +99,5 @@
                 <state_interface name="temperature"/>
             </joint>
-            <joint name="${prefix}joint3">
+            <joint name="joint3">
                 <param name="id">3</param>
                 <param name="type">vel</param>
@@ -90,5 +122,5 @@
                  this file is what a new user copies first. See the bench description under
                  test/hil/descriptions for `inverted` exercised on hardware. -->
-            <joint name="${prefix}joint4">
+            <joint name="joint4">
                 <param name="id">4</param>
                 <param name="type">vel</param>

File: description/urdf/example.urdf.xacro (robot description, xacro)
@@ -1,5 +1,10 @@
 <?xml version="1.0"?>
 <robot xmlns:xacro="http://www.ros.org/wiki/xacro" name="waveshare_servos">
-    <xacro:arg name="prefix" default="" />
+    <!-- Arguments the launch file forwards. port and baudrate are only used when
+         use_mock_hardware is false; with it true the driver is replaced by
+         mock_components/GenericSystem and no serial port is opened at all. -->
+    <xacro:arg name="port" default="/dev/ttyACM0" />
+    <xacro:arg name="baudrate" default="1000000" />
+    <xacro:arg name="use_mock_hardware" default="false" />
     <material name="white">
         <color rgba="1 1 1 1" />
@@ -14,7 +19,17 @@
         </visual>
     </link>
+    <!-- effort and velocity below are declared caps, not measured figures: 9.2 rad/s is just under
+         the servo's 6000-count goal-speed ceiling (9.2038847 rad/s) and 1.0 N m is the same cap the
+         hardware-verified bench description under test/hil declares. Keep them numerically equal to
+         the <command_interface> min/max in the ros2_control block beside this file: ros2_control
+         merges the two and enforces whichever is tighter. lower/upper are read only for revolute
+         and prismatic joints and are silently discarded for continuous ones, which is why joint3
+         and joint4 declare none - a wheel joint's position is unbounded once the driver unwraps it.
+         The <limit> element itself is kept on the wheels on purpose: a joint_trajectory_controller
+         older than 4.42.0 dereferences a null limits pointer at load time when a continuous joint
+         has none. -->
     <joint name="joint1" type="revolute">
         <axis xyz="0 0 1"/>
-        <limit effort="1000.0" lower="-1.570796" upper="1.570796" velocity="0.5"/>
+        <limit effort="1.0" lower="-1.570796" upper="1.570796" velocity="9.2"/>
         <origin xyz="0 0 0.3"/>
         <parent link="base_link"/>
@@ -32,5 +47,5 @@
     <joint name="joint2" type="revolute">
         <axis xyz="1 0 0"/>
-        <limit effort="1000.0" lower="-1.570796" upper="1.570796" velocity="0.5"/>
+        <limit effort="1.0" lower="-1.570796" upper="1.570796" velocity="9.2"/>
         <origin rpy="0 0 0" xyz="0 0 0.3"/>
         <parent link="link2"/>
@@ -48,5 +63,5 @@
     <joint name="joint3" type="continuous">
         <axis xyz="0 0 1"/>
-        <limit effort="1000.0" lower="-3.14" upper="3.14" velocity="1.0"/>
+        <limit effort="1.0" velocity="9.2"/>
         <origin xyz="0 0 0.3"/>
         <parent link="link3"/>
@@ -66,5 +81,5 @@
     <joint name="joint4" type="continuous">
         <axis xyz="0 0 1"/>
-        <limit effort="1000.0" lower="-3.14" upper="3.14" velocity="1.0"/>
+        <limit effort="1.0" velocity="9.2"/>
         <origin xyz="0 0 0.1"/>
         <parent link="link4"/>
@@ -81,4 +96,7 @@
     </link>
     <xacro:include filename="$(find waveshare_servos)/description/ros2_control/example.ros2_control.xacro"/>
-    <xacro:example_ws_ros2_control name="example_ws_ros2_control" prefix="$(arg prefix)"/>
+    <xacro:example_ws_ros2_control name="example_ws_ros2_control"
+                                   port="$(arg port)"
+                                   baudrate="$(arg baudrate)"
+                                   use_mock_hardware="$(arg use_mock_hardware)"/>
 </robot>
