Commit message: update docs and comments

File: description/ros2_control/example.ros2_control.xacro (robot description, xacro)
@@ -3,42 +3,14 @@
     <xacro:macro name="example_ws_ros2_control"
                  params="name port:=/dev/ttyACM0 baudrate:=1000000 use_mock_hardware:=false">
-        <!-- use_mock_hardware accepts true, false, 1 or 0, in any case and with any surrounding
-             space. The list lookup is deliberate: an unrecognised spelling raises inside xacro and
-             aborts the render with exit 2 ("'yes' is not in list"), which aborts the launch. A
-             plain string comparison against 'true' would treat use_mock_hardware:=yes as false and
-             quietly open the real serial port instead. -->
+        <!-- true/false/1/0 in any case. Any other value aborts the render (exit 2), so a typo
+             such as 'yes' cannot silently open the real port. -->
         <xacro:property name="mock"
             value="${['false', '0', 'true', '1'].index(str(use_mock_hardware).strip().lower()) >= 2}"/>
-        <!-- Optional, ros2_control 4.48 - read and write the hardware at its own rate, and/or on
-             its own thread. Both are ATTRIBUTES of this element, not <param> children of
-             <hardware>, and an attribute the parser does not know is dropped without a word, so a
-             typo looks like nothing happened. Pick an rw_rate that divides the update_rate: at
-             update_rate 100, rw_rate 60 is reported by `ros2 control list_hardware_components` as
-             60 Hz and actually runs at 50, while 0 or anything above update_rate is silently
-             treated as update_rate. /joint_states keeps publishing at update_rate either way - a
-             lower rw_rate does not slow the topic down, it makes each value repeat. This package
-             sets neither: rw_rate 50 halves bus occupancy but fails this package's own velocity
-             gate on a wheel near 2 rad/s, and is_async changed no measurable number at four
-             servos. See the README, "Running the bus slower, or off the control thread". To use
-             one, add the attribute to the live tag below; this copy is only the shape, and xacro
-             does not expand anything inside a comment.
-        <ros2_control name="..." type="system" rw_rate="50" is_async="true">
-        -->
+        <!-- Optional attributes of this tag, such as rw_rate="50" is_async="true"; the parser
+             drops a misspelt one silently. See docs/bus-timing.md, "rw_rate and is_async". -->
         <ros2_control name="${name}" type="system">
             <hardware>
-                <!-- use_mock_hardware:=true swaps the driver for ros2_control's own loopback
-                     simulator, which ships inside hardware_interface, opens no serial port and
-                     mirrors every command straight back into its matching state. The four <joint>
-                     blocks below are shared verbatim with the real driver: GenericSystem ignores
-                     the id/type/offset params it does not know, and a state interface with no
-                     command interface (effort, temperature) simply reads a constant 0.0. Two mock
-                     behaviours are not bugs: a velocity-commanded joint's position state never
-                     advances, so joint3 and joint4 stand still in RViz and the diff_drive odometry
-                     stays at zero; and nothing validates port, baudrate or id, so a green mock run
-                     says nothing about your wiring. The obvious cure for the frozen wheel position
-                     - the calculate_dynamics param - is a trap: it rejects any joint claiming two
-                     of position/velocity/acceleration, which is exactly what
-                     joint_trajectory_position_controller does to joint1 and joint2, and that
-                     controller then fails to activate. Do not add it. -->
+                <!-- Mock hardware opens no port, and wheel positions stay at zero; do not
+                     add calculate_dynamics. See docs/setup.md, "Try it without hardware". -->
                 <xacro:if value="${mock}">
                     <plugin>mock_components/GenericSystem</plugin>
@@ -48,24 +20,10 @@
                     <param name="port">${port}</param>
                     <param name="baudrate">${baudrate}</param>
-                    <!-- Optional, shown with their defaults and deliberately left out so this
-                         example exercises them -
-                         io_timeout_ms 5, ping_attempts 3, max_read_fails 50,
-                         allow_missing_servos false, protocol sms_sts, feedback_mode auto,
-                         encoder_steps 4096, current_per_count_a 0.006,
-                         torque_constant_nm_per_a 0.8825985. Each is described in the README,
-                         "Hardware parameters". -->
+                    <!-- The other hardware params keep their defaults on purpose.
+                         See docs/configuration.md, "Hardware parameters". -->
                 </xacro:unless>
             </hardware>
-            <!-- State interfaces are free-form - declare any subset of position, velocity,
-                 effort, current, voltage, temperature, load and status, in any order. `torque` is
-                 a deprecated alias of `effort` that keeps reporting kg cm instead of N m.
-                 The min/max below and the <limit> tags in the URDF beside this file are MERGED,
-                 most-restrictive-wins, so keep the two numerically identical: whichever is tighter
-                 is what the framework enforces, and a disagreement makes the description behave
-                 differently depending on a controller-manager flag. They only bite when the
-                 controller manager runs with enforce_command_limits: true; this example ships with
-                 it off, and the driver clamps position commands to these same values on its own.
-                 The driver ignores the velocity min/max: a wheel's speed is bounded by its
-                 joint's max_speed (9.2039 rad/s by default). -->
+            <!-- Any subset of the state interfaces, in any order. Keep min/max equal to the URDF
+                 <limit>. See docs/configuration.md, "Command interfaces and limits". -->
             <joint name="joint1">
                 <param name="id">1</param>
@@ -114,15 +72,6 @@
                 <state_interface name="temperature"/>
             </joint>
-            <!-- The second wheel, id 4, the same shape as joint3 - the example declares four
-                 joints because the reference bench carries four servos (ids 1-4), and a
-                 three-joint example on a four-servo bus leaves one servo unread and unwritten.
-                 A mirrored wheel pair is what `inverted` exists for - the right-hand wheel of a
-                 differential drive would add <param name="inverted">true</param>, which flips its
-                 velocity command together with its position, velocity and load states, so that
-                 one positive velocity drives the pair forward. It is deliberately left off here,
-                 because the URDF beside this file is a serial chain rather than a mirrored pair,
-                 so an inverted joint4 would spin its servo opposite to the model RViz draws, and
-                 this file is what a new user copies first. See the bench description under
-                 test/hil/descriptions for `inverted` exercised on hardware. -->
+            <!-- Second wheel, id 4. No inverted param: this URDF is a serial chain, not a
+                 mirrored wheel pair. See docs/configuration.md, "Adapt the example". -->
             <joint name="joint4">
                 <param name="id">4</param>

File: description/urdf/example.urdf.xacro (robot description, xacro)
@@ -1,7 +1,6 @@
 <?xml version="1.0"?>
 <robot xmlns:xacro="http://www.ros.org/wiki/xacro" name="waveshare_servos">
-    <!-- Arguments the launch file forwards. port and baudrate are only used when
-         use_mock_hardware is false; with it true the driver is replaced by
-         mock_components/GenericSystem and no serial port is opened at all. -->
+    <!-- Arguments from the launch file. port and baudrate are ignored when use_mock_hardware
+         is true (no serial port is opened). -->
     <xacro:arg name="port" default="/dev/ttyACM0" />
     <xacro:arg name="baudrate" default="1000000" />
@@ -19,15 +18,6 @@
         </visual>
     </link>
-    <!-- effort and velocity below are declared caps, not measured figures: 9.2 rad/s is just under
-         the driver's default max_speed, 6000 steps/s (9.2038847 rad/s), and 1.0 N m is the same
-         cap the hardware-verified bench description under test/hil declares. Keep them
-         numerically equal to the <command_interface> min/max in the ros2_control block beside
-         this file: ros2_control merges the two and enforces whichever is tighter. lower/upper are
-         read only for revolute and prismatic joints and are silently discarded for continuous
-         ones, which is why joint3 and joint4 declare none - a wheel joint's position is unbounded
-         once the driver unwraps it.
-         The <limit> element itself is kept on the wheels on purpose: a joint_trajectory_controller
-         older than 4.42.0 dereferences a null limits pointer at load time when a continuous joint
-         has none. -->
+    <!-- Caps, not measured values: keep equal to the ros2_control min/max. Wheels keep <limit>,
+         without lower/upper. See docs/configuration.md, "Command interfaces and limits". -->
     <joint name="joint1" type="revolute">
         <axis xyz="0 0 1"/>

File: test/hil/descriptions/bench.urdf.xacro (robot description, xacro)
@@ -1,9 +1,5 @@
 <?xml version="1.0"?>
-<!-- The bench check's description (PHASE2_SPEC 12.5). One file with arguments, because the ten
-     scenarios differ only in allow_missing_servos, the absent servo, inverted, the two
-     per-joint limits, the two <limit> ceilings H12 tightens and whether every state interface
-     is declared.
-     joint1/joint2 are the arm servos (ids 1 and 2, pos, offset 1.570796); joint3/joint4 are the
-     wheels (ids 3 and 4, vel, unwrap explicitly true); joint5 is the deliberately absent id 9. -->
+<!-- Bench check description; the scenarios vary it through xacro arguments. joint1/2: arm,
+     ids 1, 2 (pos, offset 1.570796); joint3/4: wheels, ids 3, 4 (vel); joint5: absent id 9. -->
 <robot xmlns:xacro="http://www.ros.org/wiki/xacro" name="waveshare_bench">
   <xacro:arg name="port" default="/dev/ttyACM0"/>
@@ -17,12 +13,6 @@
   <xacro:arg name="speed4" default=""/>
   <xacro:arg name="accel4" default=""/>
-  <!-- The two <limit> values the controller manager's JointSaturationLimiter reads when
-       enforce_command_limits is on (H12 only; every other scenario leaves the limiters off and
-       never notices these). They default to the values the limits were written with, so only H12
-       renders anything different. They are arguments, and NOT the same numbers as the command
-       interface min/max below, because that separation is the whole of H12's attribution: the
-       driver clamps to the command interface min/max and to max_speed_counts and never reads a
-       URDF <limit> at all, so a command clamped at a value only the description knows can only
-       have been clamped by the limiter. See h_H12 in test/hil_check.sh. -->
+  <!-- The <limit> values the JointSaturationLimiter reads. H12 tightens them below the driver's
+       own clamps (position min/max, max_speed), so a clamp at them can only be the limiter's. -->
   <xacro:arg name="arm_pos_limit" default="1.570796"/>
   <xacro:arg name="wheel_vel_limit" default="9.2038847"/>
@@ -54,6 +44,6 @@
     <xacro:wheel_link name="joint5"/>
   </xacro:if>
-  <!-- With nine:=true every interface of PHASE2_SPEC 7.2 is declared, in that order, the
-       deprecated torque alias included (H9). Otherwise the six H7 needs are declared. -->
+  <!-- nine:=true declares all nine state interfaces, the deprecated torque included (H9);
+       otherwise the six that H7 needs. -->
   <xacro:macro name="states">
     <state_interface name="position"/>
